File: test1.kicad_pcb (KiCad board)
At the start: 2 copper layers, 34.3 x 48.3 mm, 7 parts, among them IC1 ATMEGA328P-P, P1 CONN_01X02, Y1 16MHz

Commit message: Changes to schematic and PCB
Parts:
- added D1: LED, LEDs:LED-5MM, F.Cu at (222.2, 85.1)
- added D2: IR, LEDs:LED-5MM, F.Cu at (232.4, 83.8)
- added D3: IR, LEDs:LED-5MM, F.Cu at (242.6, 81.3)
- added D4: LED, LEDs:LED-5MM, F.Cu at (219.7, 97.8)
- added D5: LED, LEDs:LED-5MM, F.Cu at (232.4, 91.4)
- added D6: LED, LEDs:LED-5MM, F.Cu at (248.9, 94.0)
- added D7: LED, LEDs:LED-5MM, F.Cu at (232.4, 102.9)
- added P2: CONN_01X03, Pin_Headers:Pin_Header_Straight_1x03, F.Cu at (243.8, 119.4)
- added P3: CONN_01X03, Pin_Headers:Pin_Header_Straight_1x03, F.Cu at (259.1, 121.9)
- added P4: CONN_01X02, Pin_Headers:Pin_Header_Straight_1x02, F.Cu at (243.8, 135.9)
- added P5: CONN_01X06, Pin_Headers:Pin_Header_Straight_1x06, F.Cu at (208.3, 82.5)
- added P6: CONN_01X02, Pin_Headers:Pin_Header_Straight_1x02, F.Cu at (256.5, 135.9)
- added P7: CONN_01X02, Pin_Headers:Pin_Header_Straight_1x02, F.Cu at (247.7, 143.5)
- added P8: CONN_01X01, Connect:1pin, F.Cu at (242.6, 106.7)
- added P9: CONN_01X01, Connect:1pin, F.Cu at (251.5, 104.1)
- added R1: 330R, Resistors_ThroughHole:Resistor_Horizontal_RM10mm, F.Cu at (199.4, 130.8)
- added R10: 10k, Resistors_ThroughHole:Resistor_Horizontal_RM10mm, F.Cu at (212.1, 121.9)
- added R2: 10k, Resistors_ThroughHole:Resistor_Horizontal_RM10mm, F.Cu at (208.3, 151.1)
- added R3: 10k, Resistors_ThroughHole:Resistor_Horizontal_RM10mm, F.Cu at (167.6, 134.6)
- added R4: 330R, Resistors_ThroughHole:Resistor_Horizontal_RM10mm, F.Cu at (151.1, 141.0)
- added R5: 330R, Resistors_ThroughHole:Resistor_Horizontal_RM10mm, F.Cu at (149.9, 151.1)
- added R6: 330R, Resistors_ThroughHole:Resistor_Horizontal_RM10mm, F.Cu at (168.9, 156.2)
- added R7: 330R, Resistors_ThroughHole:Resistor_Horizontal_RM10mm, F.Cu at (221.0, 133.3)
- added R8: 10k, Resistors_ThroughHole:Resistor_Horizontal_RM10mm, F.Cu at (201.9, 139.7)
- added R9: 10k, Resistors_ThroughHole:Resistor_Horizontal_RM10mm, F.Cu at (219.7, 146.1)
- added SW1: SW_PUSH_SMALL_H, Buttons_Switches_ThroughHole:SW_PUSH_6mm_h5mm, F.Cu at (194.3, 148.6)
- moved C1 72.2 mm to (117.8, 86.9)
- moved C2 72.2 mm to (96.2, 81.8)
- moved C3 72.2 mm to (96.2, 104.7)
- moved C4 72.2 mm to (117.8, 90.7)
- moved IC1 72.2 mm to (106.3, 71.3)
- moved P1 72.2 mm to (96.2, 66.6)
- moved Y1 72.2 mm to (98.8, 93.3)
Connections:
- IC1 pad 1: Net-(IC1-Pad1) -> nRST
- IC1 pad 12: Net-(IC1-Pad12) -> WHISKER_L
- IC1 pad 13: Net-(IC1-Pad13) -> WHISKER_R
- IC1 pad 15: Net-(IC1-Pad15) -> MTR_PWM_1
- IC1 pad 16: Net-(IC1-Pad16) -> MTR_PWM_2
- IC1 pad 23: Net-(IC1-Pad23) -> PHOTO_ADC1
- IC1 pad 24: Net-(IC1-Pad24) -> PHOTO_ADC2
- IC1 pad 4: Net-(IC1-Pad4) -> LED3
- IC1 pad 5: Net-(IC1-Pad5) -> LED2
- IC1 pad 6: Net-(IC1-Pad6) -> LED1
Routing:
- net (no net): track 0.00 -> 41.5 mm
- net Net-(C3-Pad2): track 16.4 -> 0.00 mm
- net Net-(C2-Pad2): track 16.1 -> 0.00 mm
- net Net-(C1-Pad1): track 4.78 -> 0.00 mm
- net +5V: track 39.4 -> 35.2 mm
Other:
- board size 34.3 x 48.3 mm -> 100 x 100 mm
