File: test1.sch (KiCad schematic (older format))
At the start: 7 parts, among them IC1 ATMEGA328P-P, P1 CONN_01X02, Y1 16MHz

Commit message: Adding some extra components
Parts:
- added D1, D4, D5, D6, D7: LED, symbol LED
- added D2, D3: D_Small, symbol D_Small
- added P2, P3: CONN_01X03, symbol CONN_01X03
- added R1, R2, R3, R4, R5, R6, R7: R, symbol R
Connections:
- net +5V: now also D2.1 (K), D3.1 (K), P2.3 (P3), P3.3 (P3), R1.1, R4.1
- net GND: now also D1.1 (K), D4.1 (K), D5.1 (K), D6.1 (K), D7.1 (K), P2.1 (P1), P3.1 (P1), R2.2, R3.2
- net MTR_PWM_1: now reaches IC1.15 ((PCINT1/OC1A)PB1)
- net MTR_PWM_1: now also P2.2 (P2)
- net MTR_PWM_2: now reaches IC1.16 ((PCINT2/OC1B/~SS~)PB2)
- net MTR_PWM_2: now also P3.2 (P2)
- net PHOTO_ADC1: now reaches IC1.23 ((PCINT8/ADC0)PC0)
- net PHOTO_ADC1: now also D2.2 (A), R2.1
- net PHOTO_ADC2: now reaches IC1.24 ((PCINT9/ADC1)PC1)
- net PHOTO_ADC2: now also D3.2 (A), R3.1
- net LED3: now reaches IC1.4 ((PCINT18/INT0)PD2)
- net LED3: now also R5.1
- net LED2: now reaches IC1.5 ((PCINT19/OC2B/INT1)PD3)
- net LED2: now also R6.1
- net LED1: now reaches IC1.6 ((PCINT20/XCK/T0)PD4)
- net LED1: now also R7.1
- new net: D1.2 (A), R1.2
- new net: D4.2 (A), R4.2
- new net: D5.2 (A), R5.2
- new net: D6.2 (A), R6.2
- new net: D7.2 (A), R7.2
- no-connect marks 21 -> 14
Other:
- note added: "IR Left/Right Transmitters"
- note added: "IR receivers left/right"
- note added: "Indication LEDs"
- note added: "Motor drivers"
- note added: "Power connector"
- moved on the sheet: C1, C2, C3, C4, IC1, P1, Y1

Commit message: Changes to schematic and PCB
Parts:
- removed Y1: 16MHz, Crystals:Crystal_HC48-U_Vertical, symbol Crystal
- added P4: CONN_01X02, Pin_Headers:Pin_Header_Straight_1x02, symbol CONN_01X02
- added P5: CONN_01X06, symbol CONN_01X06
- added P6, P7: CONN_01X02, symbol CONN_01X02
- added P8, P9: CONN_01X01, symbol CONN_01X01
- added R10, R8, R9: 10k, symbol R
- added SW1: SW_PUSH_SMALL_H, symbol SW_PUSH_SMALL_H
- added Y1: 16MHz, symbol Crystal_Small
- D2, D3: value D_Small -> IR
- R1, R4, R5, R6, R7: value R -> 330R
- R2, R3: value R -> 10k
Connections:
- net +5V: now also P5.2 (P2), R10.1, R8.1, R9.1
- net GND: now also P5.6 (P6), P8.1 (P1), P9.1 (P1), SW1.2
- net nRST: now reaches IC1.1 ((PCINT14/~RESET~)PC6)
- net nRST: now also P5.5 (P5), R8.2, SW1.1
- net at C3.2, IC1.10 ((PCINT7/XTAL2/TOSC2)PB7): now also Y1.2
- net WHISKER_L: now reaches IC1.12 ((PCINT22/OC0A/AIN0)PD6)
- net WHISKER_L: now also P6.1 (P1), P6.2 (P2), R9.2
- net WHISKER_R: now reaches IC1.13 ((PCINT23/AIN1)PD7)
- net WHISKER_R: now also P7.1 (P1), P7.2 (P2), R10.2
- net at IC1.17 ((PCINT3/OC2A/MOSI)PB3): now also P5.4 (P4)
- net at IC1.18 ((PCINT4/MISO)PB4): now also P5.1 (P1)
- net at IC1.19 ((PCINT5/SCK)PB5): now also P5.3 (P3)
- net at IC1.2 ((PCINT16/RXD)PD0): now also P4.1 (P1)
- net at IC1.3 ((PCINT17/TXD)PD1): now also P4.2 (P2)
- net at C2.2, IC1.9 ((PCINT6/XTAL1/TOSC1)PB6): now also Y1.1
- no-connect marks 14 -> 6
Other:
- note added: "ICSP"
- note added: "Program"
- note added: "Whiskers"
- moved on the sheet: C1, C2, C3, C4, IC1, P2, P3
