File: botuino.sch (KiCad schematic (older format))
At the start: 62 parts, among them IC1 ATMEGA328P-P, P1 CONN_01X02, P10 CONN_01X03, P11 CONN_01X01, P12 CONN_01X01, P13 CONN_01X01, P14 CONN_01X01, P15 CONN_01X01, P16 CONN_01X01, P17 CONN_01X01, P18 CONN_01X01, P19 CONN_01X01, P2 CONN_01X03, P20 CONN_01X01, P21 CONN_01X01, P22 CONN_01X01, P23 CONN_01X01, P24 CONN_01X01, P25 CONN_01X01, P26 CONN_01X01, P27 CONN_01X01, P3 CONN_01X03, P4 CONN_01X03, P5 CONN_01X06, P6 CONN_01X02, P7 CONN_01X02, P8 CONN_01X01, P9 CONN_01X01, Q1 BC546, Y1 16MHz

Commit message: Updating schematic with title and version number
Other:
- note added: "1 1"
- note added: "22/01/2017"
- note added: "v1.0"
Changed lines of the file:
@@
 EESchema Schematic File Version 2
-LIBS:test1-rescue
 LIBS:power
 LIBS:device
@@
 F 0 "Q1" H 5850 7175 50  0000 L CNN
 F 1 "BC546" H 5850 7100 50  0000 L CNN
-F 2 "TO_SOT_Packages_THT:TO-92_Inline_Narrow_Oval" H 5850 7025 50  0000 L CIN
+F 2 "TO_SOT_Packages_THT:TO-92_Inline_Narrow_Oval" H 3950 6750 50  0000 L CIN
 F 3 "" H 5650 7100 50  0000 L CNN
 	1    5650 7100
@@
 Wire Wire Line
 	5750 6900 5750 6800
+Text Notes 7300 7250 0    60   ~ 0
+1 1
+Text Notes 7500 7500 0    60   ~ 0
+Botuino
+Text Notes 8200 7650 0    60   ~ 0
+22/01/2017
+Text Notes 10650 7650 0    60   ~ 0
+v1.0
 $EndSCHEMATC
